File: pcb files/ledCubeV2.0.sch (EAGLE design)
At the start: 225 parts, among them IC1 74HC02D, IC2 74HC02D, IC3 74AHC1G08DCK, Q1 BSS84, Q2 BSS123, T1 PMBT3904, T2 PMBT3904, U1 ESP12-E

Commit message: Update ledCubeV2.0.sch
Other:
- note removed: "WRONG TRANSISTOR PINOUT!!"
